File: Kicad/Trackball/Trackball.kicad_pcb (KiCad board)
At the start: 2 copper layers, 410.3 x 138.1 mm, 67 parts, among them J1 Battery, J10 Conn_01x04_Female, J12 Conn_01x04_Female, J13 Conn_01x04_Female, J15 Conn_01x04_Female, J18 Conn_01x03_Pin, J19 Conn_01x03_Pin, J2 Conn_01x04_Male, J20 Conn_01x03_Socket, J21 Conn_01x03_Socket, J3 Conn_01x04_Male, J4 Conn_01x04_Male, J5 Conn_01x04_Male, SW1 SW_SPDT, SW2 SW_SPDT, SW3 SW_SPDT, U1 ProMicro, U3 TCR2EF19, U4 PMW3610

Commit message: B4: Corrected the PCBs, added two more keys. TODO: add 55mm top deck.
Parts:
- added MX10: MX-NoLED, keyswitches.pretty-master:Kailh_socket_PG1350, F.Cu at (248.0, 89.1)
- added MX11: MX-NoLED, keyswitches.pretty-master:Kailh_socket_PG1350, F.Cu at (379.9, 89.1)
- added MX12: MX-NoLED, keyswitches.pretty-master:Kailh_socket_PG1350, F.Cu at (379.8, 114.1)
- added MX9: MX-NoLED, keyswitches.pretty-master:Kailh_socket_PG1350, F.Cu at (248.0, 114.1)
- moved J1 4.86 mm to (136.0, 87.7), turned to 45 degrees
- moved H12 3.00 mm to (165.4, 143.6)
- moved H13 3.00 mm to (165.4, 59.6)
- moved H2 3.00 mm to (60.4, 143.6)
- moved H8 3.00 mm to (60.2, 59.6)
- moved J12 3.00 mm to (168.8, 126.0)
- moved J15 3.00 mm to (168.8, 77.2)
- moved J6 3.00 mm to (388.6, 126.0)
- moved J7 3.00 mm to (388.6, 77.2)
- moved MX1 3.00 mm to (248.0, 138.7), turned to 0 degrees
- moved MX4 3.00 mm to (248.0, 64.4), turned to 180 degrees
- moved MX7 3.00 mm to (379.8, 138.7), turned to 0 degrees
- moved MX8 3.00 mm to (379.8, 64.4), turned to 180 degrees
- moved J4 3.00 mm to (256.8, 126.0)
- moved J5 3.00 mm to (256.8, 77.2)
- renumbered H6 to H17, H4 to H18, H3 to H19, H5 to H20, H7 to H21, H1 to H22, J4 to J6, J5 to J7, J3 to J8, J2 to J9, MX1 to MX7, MX4 to MX8
Connections:
- H17 pad 1: GNDA -> GNDC
- H18 pad 1: GNDA -> GNDC
- H19 pad 1: GNDA -> GNDC
- H20 pad 1: GNDA -> GNDC
- H21 pad 1: GNDA -> GNDC
- H22 pad 1: GNDA -> GNDC
- J12 pad 1: GND -> Button7
- J15 pad 1: GND -> Button8
- J4 pad 1: GNDA -> Net-(J4-Pin_1)
- J5 pad 2: Net-(J5-Pin_1) -> GNDA
- J5 pad 3: Net-(J5-Pin_1) -> GNDA
- J6 pad 1: GNDA -> Net-(J6-Pin_1)
- J6 pad 2: GNDA -> GNDC
- J6 pad 3: GNDA -> GNDC
- J6 pad 4: Net-(J4-Pin_4) -> Net-(J6-Pin_4)
- J7 pad 1: Net-(J5-Pin_1) -> Net-(J7-Pin_1)
- J7 pad 2: Net-(J5-Pin_1) -> GNDC
- J7 pad 3: Net-(J5-Pin_1) -> GNDC
- J7 pad 4: Net-(J5-Pin_4) -> Net-(J7-Pin_4)
- J8 pad 1: GNDA -> GNDC
- J8 pad 2: GNDA -> GNDC
- J8 pad 3: GNDA -> GNDC
- J8 pad 4: GNDA -> GNDC
- J9 pad 1: GNDA -> GNDC
- J9 pad 2: GNDA -> GNDC
- J9 pad 3: GNDA -> GNDC
- J9 pad 4: GNDA -> GNDC
- MX7 pad 1: Net-(J4-Pin_4) -> Net-(J6-Pin_4)
- MX7 pad 2: GNDA -> GNDC
- MX8 pad 1: GNDA -> GNDC
- MX8 pad 2: Net-(J5-Pin_4) -> Net-(J7-Pin_4)
- U1 pad 17: unconnected-(U1-F7-Pad17) -> Button8
- U1 pad 18: unconnected-(U1-F6-Pad18) -> Button7
Routing:
- net Button7: track 0.00 -> 47.6 mm, vias 0 -> 1
- net Net-(J1-Pin_1): track 0.00 -> 40.7 mm
- net Button8: track 0.00 -> 36.9 mm, vias 0 -> 1
- net Net-(J6-Pin_4): track 0.00 -> 23.9 mm
- net Net-(J7-Pin_1): track 0.00 -> 23.5 mm
- net Net-(J5-Pin_1): track 0.00 -> 22.4 mm
- net Net-(J7-Pin_4): track 0.00 -> 19.5 mm
- net Net-(J6-Pin_1): track 0.00 -> 17.4 mm
- net Net-(J4-Pin_1): track 0.00 -> 16.3 mm
- net Net-(J5-Pin_4): track 31.0 -> 19.5 mm
- net BTReset: track 39.9 -> 47.7 mm
- net Handiness: track 11.8 -> 18.4 mm
- net Button4: track 39.8 -> 45.6 mm
- net Net-(J1-Pin_2): track 44.4 -> 39.5 mm
- net NCS: track 40.3 -> 43.9 mm
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- added copper zone on B.Cu, net GNDC
- added copper zone on F.Cu, net GNDC
Other:
- board size 410.3 x 138.1 mm -> 413.3 x 138.1 mm

Commit message: B4: Added 55mm top PCB, moved the buttons  around, reduced the overall outline. TODO: lay out the wiring.
Parts:
- added H23: MountingHole_Pad, MountingHole:MountingHole_2.5mm_Pad, F.Cu at (411.6, 82.2)
- added H24: MountingHole_Pad, MountingHole:MountingHole_2.5mm_Pad, F.Cu at (411.6, 121.1)
- added H25: MountingHole_Pad, MountingHole:MountingHole_2.5mm_Pad, F.Cu at (389.2, 82.2)
- added H26: MountingHole_Pad, MountingHole:MountingHole_2.5mm_Pad, F.Cu at (377.9, 101.6)
- added J11: Conn_01x04_Male, Connector_PinHeader_2.54mm:PinHeader_1x04_P2.54mm_Vertical, B.Cu at (349.7, 97.8)
- added J14: Conn_01x04_Female, Connector_PinSocket_2.54mm:PinSocket_1x04_P2.54mm_Vertical, F.Cu at (176.9, 97.8)
- added J16: Conn_01x04_Male, Connector_PinHeader_2.54mm:PinHeader_1x04_P2.54mm_Vertical, B.Cu at (264.9, 97.8)
- added J17: Conn_01x04_Male, Connector_PinHeader_2.54mm:PinHeader_1x04_P2.54mm_Vertical, B.Cu at (382.6, 122.8)
- added J22: Conn_01x04_Male, Connector_PinHeader_2.54mm:PinHeader_1x04_P2.54mm_Vertical, B.Cu at (446.6, 126.0)
- added J23: Conn_01x04_Male, Connector_PinHeader_2.54mm:PinHeader_1x04_P2.54mm_Vertical, B.Cu at (446.6, 77.2)
- added J24: Conn_01x04_Male, Connector_PinHeader_2.54mm:PinHeader_1x04_P2.54mm_Vertical, B.Cu at (382.6, 80.4)
- added J25: Conn_01x04_Male, Connector_PinHeader_2.54mm:PinHeader_1x04_P2.54mm_Vertical, B.Cu at (437.7, 97.8)
- added MX13: MX-NoLED, keyswitches.pretty-master:Kailh_socket_PG1350, F.Cu at (307.6, 69.4)
- added MX14: MX-NoLED, keyswitches.pretty-master:Kailh_socket_PG1350, F.Cu at (307.6, 133.0)
- added MX15: MX-NoLED, keyswitches.pretty-master:Kailh_socket_PG1350, F.Cu at (437.8, 114.1)
- added MX16: MX-NoLED, keyswitches.pretty-master:Kailh_socket_PG1350, F.Cu at (437.8, 89.1)
- added MX17: MX-NoLED, keyswitches.pretty-master:Kailh_socket_PG1350, F.Cu at (395.5, 136.8)
- added MX18: MX-NoLED, keyswitches.pretty-master:Kailh_socket_PG1350, F.Cu at (395.5, 66.4)
- added MX19: MX-NoLED, keyswitches.pretty-master:Kailh_socket_PG1350, F.Cu at (437.8, 138.8)
- added MX20: MX-NoLED, keyswitches.pretty-master:Kailh_socket_PG1350, F.Cu at (437.8, 64.4)
- H10, H15: footprint MountingHole:MountingHole_3.7mm_Pad -> MountingHole:MountingHole_2.5mm_Pad
- moved H10 440.8 mm to (423.0, 101.6)
- moved H15 302.4 mm to (389.2, 121.0)
- moved MX3 102.3 mm to (222.7, 136.7), turned to 0 degrees
- moved MX6 102.3 mm to (222.7, 66.4), turned to 180 degrees
- moved H11 43.0 mm to (40.2, 69.1)
- moved H9 43.0 mm to (40.1, 134.1)
- moved J1 38.5 mm to (172.4, 75.1), turned to -90 degrees
- moved H8 33.4 mm to (92.2, 69.1)
- moved H2 33.4 mm to (92.4, 134.2)
- moved H19 30.0 mm to (332.1, 101.7)
- moved J6 30.0 mm to (358.6, 126.0)
- moved J7 30.0 mm to (358.6, 77.2)
- moved MX12 30.0 mm to (349.8, 114.1)
- moved MX7 30.0 mm to (349.8, 138.7), turned to 90 degrees
- moved MX8 30.0 mm to (349.8, 64.4), turned to 90 degrees
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Connections:
- H10 pad 1: GNDB -> GNDE
- H15 pad 1: GND -> GNDE
- J12 pad 3: GND -> Button3
- J15 pad 3: GND -> Button6
- J4 pad 3: GNDA -> Net-(J4-Pin_3)
- J5 pad 3: GNDA -> Net-(J5-Pin_3)
- J6 pad 3: GNDC -> Net-(J6-Pin_3)
- J7 pad 3: GNDC -> Net-(J7-Pin_3)
- MX3 pad 1: GND -> Net-(J4-Pin_3)
- MX3 pad 2: Button3 -> GNDA
- MX5 pad 1: Button5 -> GND
- MX5 pad 2: GND -> Button5
- MX6 pad 1: Button6 -> GNDA
- MX6 pad 2: GND -> Net-(J5-Pin_3)
Routing:
- net Button3: track 52.6 -> 0.00 mm, vias 2 -> 0
- net Net-(J1-Pin_1): track 40.7 -> 0.00 mm
- net Net-(J1-Pin_2): track 39.5 -> 0.00 mm, vias 1 -> 0
- net Unlock: track 58.9 -> 30.8 mm
- net Button6: track 66.9 -> 43.9 mm, vias 2 -> 1
- net BTReset: track 47.7 -> 24.8 mm
- net Net-(J23-Pin_1): track 0.00 -> 22.4 mm
- net Net-(J22-Pin_4): track 0.00 -> 19.6 mm
- net Net-(J5-Pin_4): track 19.5 -> 0.00 mm
- net BTSelect: track 48.1 -> 29.2 mm, vias 2 -> 1
- net Net-(J22-Pin_1): track 0.00 -> 16.3 mm
- added copper zone on B.Cu, net GNDE
- added copper zone on F.Cu, net GNDE
Other:
- board size 413.3 x 138.1 mm -> 429.8 x 138.1 mm
- board text added: "BT SEL"
- board text added: "ProMicro here FACE UP"
- board text added: "ZMK STUDIO UNLOCK"
- board text added: "u/ak66666 ThumbsUp! Trackball v4 55mm Ball"
- board text removed: "BT SELECT"
- board text removed: "ProMicro here face down"
- board text removed: "ProMicro on the other side FACE DOWN"
- board text removed: "ZMK.STUDIO UNLOCK"
